File: LED Flasher/LED Flasher.kicad_sch (KiCad schematic)
At the start: 20 parts, among them Q1 BC848, Q2 BC848, Q3 BC858, Q4 SI2342DS-T1-GE3

Commit message: Ding Dong Doorbell Project
Parts:
- Q4: value SI2342DS-T1-GE3 -> SI2338DS
Changed lines of the file:
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@@
       (effects (font (size 1.524 1.524)) (justify left))
     )
-    (property "Value" "SI2342DS-T1-GE3" (at 241.3 74.93 0)
+    (property "Value" "SI2338DS" (at 241.3 74.93 0)
       (effects (font (size 1.524 1.524)) (justify left))
     )

Commit message: Updates and improvements to LED Flasher
Parts:
- removed C1: 2.2UF-1206-50V-10%, Capacitor_SMD:C_1206_3216Metric, symbol SparkFun-Capacitors:2.2UF-1206-50V-10%
- added C1: 100UF-1210-50V-20%, Capacitor_SMD:C_1210_3225Metric, symbol SparkFun-Capacitors:10UF-1210-50V-20%
- C2: value 10UF-1210-50V-20% -> 100UF-1210-50V-20%
- R1, R4: value 15R -> 51R
Connections:
- net LED 2: now also C1.2
- net at Q1.3 (C), R1.1: now also C1.1
Changed lines of the file:
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@@
       (effects (font (size 1.143 1.143)))
     )
-    (property "Value" "10UF-1210-50V-20%" (at 130.81 69.85 90)
+    (property "Value" "100UF-1210-50V-20%" (at 130.81 69.85 90)
       (effects (font (size 1.143 1.143)))
     )
@@
     )
   )
+  (symbol (lib_id "SparkFun-Capacitors:10UF-1210-50V-20%") (at 105.41 76.2 90) (unit 1)
+    (in_bom yes) (on_board yes) (dnp no) (fields_autoplaced)
+    (property "Reference" "C1" (at 104.14 67.31 90)
+      (effects (font (size 1.143 1.143)))
+    )
+    (property "Value" "100UF-1210-50V-20%" (at 104.14 69.85 90)
+      (effects (font (size 1.143 1.143)))
+    )
+    (property "Footprint" "Capacitor_SMD:C_1210_3225Metric" (at 99.06 76.2 0)
+      (effects (font (size 0.508 0.508)) hide)
+    )
+    (property "Datasheet" "" (at 105.41 76.2 0)
+      (effects (font (size 1.27 1.27)) hide)
+    )
+    (property "Field4" "CAP-09824" (at 104.14 72.39 90)
+      (effects (font (size 1.524 1.524)))
+    )
+    (pin "1")
+    (pin "2")
+    (instances
+      (project "LED Flasher"
+        (path "/eb37c1ca-22d8-46d0-987a-ab0389058c2f"
+          (reference "C1") (unit 1)
+        )
+      )
+    )
+  )
   (symbol (lib_id "Transistor_BJT:BC848") (at 93.98 85.09 0) (unit 1)
     (in_bom yes) (on_board yes) (dnp no) (fields_autoplaced)
@@
       (effects (font (size 1.143 1.143)) (justify right))
     )
-    (property "Value" "15R" (at 142.24 60.96 90)
+    (property "Value" "51R" (at 142.24 60.96 90)
       (effects (font (size 1.143 1.143)) (justify right))
     )
@@
       (effects (font (size 1.143 1.143)) (justify right))
     )
-    (property "Value" "15R" (at 91.44 60.96 90)
+    (property "Value" "51R" (at 91.44 60.96 90)
       (effects (font (size 1.143 1.143)) (justify right))
     )
@@
         )
       )
-    )
-  )
-  (symbol (lib_id "SparkFun-Capacitors:2.2UF-1206-50V-10%") (at 105.41 76.2 90) (unit 1)
-    (in_bom yes) (on_board yes) (dnp no) (fields_autoplaced)
-    (property "Reference" "C1" (at 104.14 67.31 90)
-      (effects (font (size 1.143 1.143)))
-    )
-    (property "Value" "2.2UF-1206-50V-10%" (at 104.14 69.85 90)
-      (effects (font (size 1.143 1.143)))
-    )
-    (property "Footprint" "Capacitor_SMD:C_1206_3216Metric" (at 99.06 76.2 0)
-      (effects (font (size 0.508 0.508)) hide)
-    )
-    (property "Datasheet" "" (at 105.41 76.2 0)
-      (effects (font (size 1.27 1.27)) hide)
-    )
-    (property "Field4" "CAP-10009" (at 104.14 72.39 90)
-      (effects (font (size 1.524 1.524)))
-    )
-    (pin "1")
-    (pin "2")
-    (instances
-      (project "LED Flasher"
-        (path "/eb37c1ca-22d8-46d0-987a-ab0389058c2f"
-          (reference "C1") (unit 1)
-        )
-      )
