File: Ding Dong Doorbell/Ding Dong Doorbell.kicad_pcb (KiCad board)
At the start: 2 copper layers, 76.1 x 35.5 mm, 25 parts, among them J1 Speaker, J2 Ringer, Q1 BC848, Q2 SI2338DS, U1 NE555D

Commit message: Some Updates
Parts:
- C3: footprint Capacitors:1206 -> Capacitors:1210
- C5: footprint Capacitor_SMD:C_1206_3216Metric -> Capacitor_SMD:C_1210_3225Metric
- moved C5 0.33 mm to (147.4, 96.5)
- moved C3 0.05 mm to (117.2, 86.1)
