File: Ding Dong Doorbell/Ding Dong Doorbell.kicad_sch (KiCad schematic)
At the start: 25 parts, among them J1 Speaker, J2 Ringer, Q1 BC848, Q2 SI2338DS, U1 NE555D

Commit message: Some Updates
Parts:
- C3: footprint Capacitors:1206 -> Capacitors:1210
- C5: footprint Capacitor_SMD:C_1206_3216Metric -> Capacitor_SMD:C_1210_3225Metric
Changed lines of the file:
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@@
       (effects (font (size 1.143 1.143)) (justify left))
     )
-    (property "Footprint" "Capacitors:1206" (at 153.67 85.09 0)
+    (property "Footprint" "Capacitors:1210" (at 153.67 85.09 0)
       (effects (font (size 0.508 0.508)) hide)
     )
@@
       (effects (font (size 1.143 1.143)) (justify right))
     )
-    (property "Footprint" "Capacitor_SMD:C_1206_3216Metric" (at 224.79 80.01 0)
-      (effects (font (size 0.508 0.508)) hide)
-    )
+    (property "Footprint" "Capacitor_SMD:C_1210_3225Metric" (at 224.79 80.01 0)
+      (effects (font (size 0.508 0.508)) hide)
+    )
