File: Universal Timer/Universal Timer.kicad_sch (KiCad schematic)
At the start: 37 parts, among them J1 Timer Start, J2 Relay Out, J3 Buzz Enable, J4 On/Off, Q1 BC858, Q2 BC848, Q3 BC848, Q3 BC858, Q4 DMN2004K-7, Q4 SI2338DS, Q5 DMN2004K-7, Q8 BC848, U1 NE555D

Commit message: Backups Update
Parts:
- removed J3: Buzz Enable, Connector_PinSocket_2.54mm:PinSocket_1x02_P2.54mm_Vertical, symbol Connector:Conn_01x02_Pin
- removed LS1: ABI-009-RC, ABI-009-RC:ABI-009_MTC, symbol ABI-009-RC:ABI-009-RC
- removed Q3: BC848, Package_TO_SOT_SMD:SOT-23, symbol Transistor_BJT:BC848
- removed R6: 10k, Resistor_SMD:R_1206_3216Metric, symbol SparkFun-Resistors:RESISTOR1206
- added D3: LD271, LED_THT:LED_D5.0mm_IRGrey, symbol LED:LD271
- added R9: 360R, Resistor_SMD:R_1206_3216Metric, symbol SparkFun-Resistors:RESISTOR1206
- renumbered Q8 to Q3
Connections:
- net 9V: now also D3.2 (A)
- net CRTGND: now also R9.1
- new net: D3.1 (K), R9.2
Other:
- moved on the sheet: J2, Q3, R12

Commit message: Completed Monophonic Organ Board
Connections:
- net CRTGND is gone; now on net GND: C1.2, C2.2, C3.2, C4.2, J1.2 (Pin_2), Q2.2 (E), Q4.3, R12.1, R2.1, R5.1, R6.2, R9.1, R9.1, U1.1 (GND)
- net GND: no longer B1.1, C3.1, Q4.2, R8.1
- new net: B1.1, C3.1, Q4.2, R8.1
Changed lines of the file:
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@@
   (junction (at 181.61 143.51) (diameter 0) (color 0 0 0 0)
   )
-  (junction (at 195.58 91.44) (diameter 0) (color 0 0 0 0)
-  )
   (junction (at 201.93 96.52) (diameter 0) (color 0 0 0 0)
   )
@@
   )
   (wire (pts (xy 151.13 73.66) (xy 151.13 82.55))
-    (stroke (width 0) (type default))
-  )
-  (wire (pts (xy 208.28 91.44) (xy 195.58 91.44))
     (stroke (width 0) (type default))
   )
@@
     )
   )
-  (global_label "CRTGND" (shape input) (at 208.28 55.88 0) (fields_autoplaced)
+  (global_label "GND" (shape input) (at 208.28 55.88 0) (fields_autoplaced)
     (effects (font (size 1.27 1.27)) (justify left))
-    (property "Intersheetrefs" "${INTERSHEET_REFS}" (at 218.6433 55.88 0)
-      (effects (font (size 1.27 1.27)) (justify left) hide)
-    )
-  )
-  (global_label "GND" (shape input) (at 208.28 91.44 0) (fields_autoplaced)
-    (effects (font (size 1.27 1.27)) (justify left))
-    (property "Intersheetrefs" "${INTERSHEET_REFS}" (at 215.1357 91.44 0)
+    (property "Intersheetrefs" "${INTERSHEET_REFS}" (at 215.1357 55.88 0)
       (effects (font (size 1.27 1.27)) (justify left) hide)
     )
@@
     )
   )
-  (global_label "CRTGND" (shape input) (at 208.28 157.48 0) (fields_autoplaced)
+  (global_label "GND" (shape input) (at 208.28 157.48 0) (fields_autoplaced)
     (effects (font (size 1.27 1.27)) (justify left))
-    (property "Intersheetrefs" "${INTERSHEET_REFS}" (at 218.6433 157.48 0)
+    (property "Intersheetrefs" "${INTERSHEET_REFS}" (at 215.1357 157.48 0)
       (effects (font (size 1.27 1.27)) (justify left) hide)
     )
