File: Monophonic Organ/Monophonic Organ.kicad_sch (KiCad schematic)
At the start: 106 parts, among them IC1 NE555DR, IC2 NE555DR, IC3 HEF4069UBT,653, IC4 LT1782CS5#TRMPBF, J1 Speaker, Q1 Si2338DS-T1-GE3, Q2 BC858, Q3 Si2338DS-T1-GE3, Q4 BC848, Q5 BC858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

Commit message: Fixed mistake on organ pcb
Parts:
- added S27: FSM4JSMATR, SamacSys_Parts:FSM4JSMATR, symbol SamacSys_Parts:FSM4JSMATR
Connections:
- net PROBE: now also S27.4
- net at R2.2, R3.1: now also S27.2
- no-connect marks 61 -> 63
Changed lines of the file:
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@@
   (junction (at 184.15 97.79) (diameter 0) (color 0 0 0 0)
   )
+  (junction (at 204.47 105.41) (diameter 0) (color 0 0 0 0)
+  )
   (junction (at 105.41 139.7) (diameter 0) (color 0 0 0 0)
   )
@@
   (junction (at 128.27 139.7) (diameter 0) (color 0 0 0 0)
   )
+  (junction (at 204.47 139.7) (diameter 0) (color 0 0 0 0)
+  )
   (junction (at 133.35 115.57) (diameter 0) (color 0 0 0 0)
   )
@@
   (no_connect (at 95.25 118.11))
   (no_connect (at 175.26 158.75))
+  (no_connect (at 201.93 118.11))
   (no_connect (at 179.07 138.43))
   (no_connect (at 179.07 118.11))
@@
   (no_connect (at 95.25 138.43))
   (no_connect (at 181.61 48.26))
+  (no_connect (at 201.93 138.43))
   (no_connect (at 163.83 118.11))
   (no_connect (at 34.29 118.11))
@@
     (stroke (width 0) (type default))
   )
-  (wire (pts (xy 19.05 101.6) (xy 194.31 101.6))
+  (wire (pts (xy 19.05 101.6) (xy 204.47 101.6))
     (stroke (width 0) (type default))
   )
@@
     (stroke (width 0) (type default))
   )
-  (wire (pts (xy 194.31 101.6) (xy 194.31 105.41))
+  (wire (pts (xy 204.47 101.6) (xy 204.47 105.41))
     (stroke (width 0) (type default))
   )
@@
     (stroke (width 0) (type default))
   )
+  (wire (pts (xy 204.47 138.43) (xy 204.47 139.7))
+    (stroke (width 0) (type default))
+  )
   (wire (pts (xy 81.28 67.31) (xy 81.28 69.85))
     (stroke (width 0) (type default))
@@
     (stroke (width 0) (type default))
   )
+  (wire (pts (xy 204.47 118.11) (xy 204.47 105.41))
+    (stroke (width 0) (type default))
+  )
   (wire (pts (xy 161.29 67.31) (xy 137.16 67.31))
     (stroke (width 0) (type default))
@@
     (stroke (width 0) (type default))
   )
-  (wire (pts (xy 196.85 139.7) (xy 199.39 139.7))
+  (wire (pts (xy 196.85 139.7) (xy 204.47 139.7))
     (stroke (width 0) (type default))
   )
@@
     (stroke (width 0) (type default))
   )
+  (wire (pts (xy 204.47 105.41) (xy 194.31 105.41))
+    (stroke (width 0) (type default))
+  )
   (wire (pts (xy 90.17 115.57) (xy 87.63 115.57))
     (stroke (width 0) (type default))
@@
     (stroke (width 0) (type default))
   )
+  (wire (pts (xy 204.47 139.7) (xy 205.74 139.7))
+    (stroke (width 0) (type default))
+  )
   (global_label "9V" (shape input) (at 269.24 24.13 0) (fields_autoplaced)
     (effects (font (size 1.27 1.27)) (justify left))
@@
     )
   )
-  (global_label "PROBE" (shape input) (at 199.39 139.7 0) (fields_autoplaced)
+  (global_label "PROBE" (shape input) (at 205.74 139.7 0) (fields_autoplaced)
     (effects (font (size 1.27 1.27)) (justify left))
-    (property "Intersheetrefs" "${INTERSHEET_REFS}" (at 208.6647 139.7 0)
+    (property "Intersheetrefs" "${INTERSHEET_REFS}" (at 215.0147 139.7 0)
       (effects (font (size 1.27 1.27)) (justify left) hide)
     )
@@
     )
   )
+  (symbol (lib_id "SamacSys_Parts:FSM4JSMATR") (at 201.93 138.43 90) (unit 1)
+    (in_bom yes) (on_board yes) (dnp no)
+    (property "Reference" "S27" (at 200.66 128.27 90)
+      (effects (font (size 1.27 1.27)) (justify right))
+    )
+    (property "Value" "FSM4JSMATR" (at 200.66 130.81 90)
+      (effects (font (size 1.27 1.27)) (justify right) hide)
+    )
+    (property "Footprint" "SamacSys_Parts:FSM4JSMATR" (at 296.85 121.92 0)
+      (effects (font (size 1.27 1.27)) (justify left top) hide)
+    )
+    (property "Datasheet" "https://datasheet.datasheetarchive.com/originals/distributors/Datasheets-DGA6/576850.pdf" (at 396.85 121.92 0)
+      (effects (font (size 1.27 1.27)) (justify left top) hide)
+    )
+    (property "Height" "" (at 596.85 121.92 0)
+      (effects (font (size 1.27 1.27)) (justify left top) hide)
+    )
+    (property "element14 Part Number" "" (at 696.85 121.92 0)
+      (effects (font (size 1.27 1.27)) (justify left top) hide)
+    )
+    (property "element14 Price/Stock" "" (at 796.85 121.92 0)
+      (effects (font (size 1.27 1.27)) (justify left top) hide)
+    )
+    (property "Manufacturer_Name" "TE Connectivity" (at 896.85 121.92 0)
+      (effects (font (size 1.27 1.27)) (justify left top) hide)
+    )
+    (property "Manufacturer_Part_Number" "FSM4JSMATR" (at 996.85 121.92 0)
+      (effects (font (size 1.27 1.27)) (justify left top) hide)
+    )
+    (pin "1")
+    (pin "2")
+    (pin "3")
+    (pin "4")
+    (instances
+      (project "Monophonic Organ"
+        (path "/2f1155ed-90ab-474a-b992-9a0b1909d860"
+          (reference "S27") (unit 1)
+        )
+      )
+    )
+  )
   (symbol (lib_id "SamacSys_Parts:NE555DR") (at 168.91 63.5 0) (unit 1)
     (in_bom yes) (on_board yes) (dnp no)
@@
   (symbol (lib_id "SparkFun-Resistors:RESISTOR1206") (at 228.6 67.31 270) (unit 1)
     (in_bom yes) (on_board yes) (dnp no)
-    (property "Reference" "R44" (at 231.14 67.31 0)
+    (property "Reference" "R44" (at 232.41 66.04 90)
       (effects (font (size 1.143 1.143)))
     )
-    (property "Value" "10k" (at 233.68 67.31 0)
+    (property "Value" "10k" (at 232.41 68.58 90)
       (effects (font (size 1.143 1.143)))
     )
@@
       (effects (font (size 1.524 1.524)) hide)
     )
-    (property "Field4" " " (at 232.41 67.31 0)
+    (property "Field4" " " (at 232.41 67.31 90)
       (effects (font (size 1.524 1.524)))
     )
@@
   (symbol (lib_id "SparkFun-Resistors:RESISTOR1206") (at 228.6 31.75 270) (unit 1)
     (in_bom yes) (on_board yes) (dnp no)
-    (property "Reference" "R43" (at 231.14 31.75 0)
+    (property "Reference" "R43" (at 232.41 30.48 90)
       (effects (font (size 1.143 1.143)))
     )
-    (property "Value" "10k" (at 233.68 31.75 0)
+    (property "Value" "10k" (at 232.41 33.02 90)
       (effects (font (size 1.143 1.143)))
     )
@@
       (effects (font (size 1.524 1.524)) hide)
     )
-    (property "Field4" " " (at 232.41 31.75 0)
+    (property "Field4" " " (at 232.41 31.75 90)
       (effects (font (size 1.524 1.524)))
     )
